Commit message: Change path pattern.

File: robotiq_2f_85_gripper_visualization/urdf/robotiq_gripper.urdf (robot description, URDF)
Before this commit: robot robotiq_gripper, 13 links, 12 joints
Links:
- link left_inner_finger: geometry collision mesh filename=file://$(find robotiq_2f_85_gripper_visualization)/meshes/c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 scale=0.001 0.001 0.001; visual mesh filename=file://$(find robotiq_2f_85_gripper_visualization)/meshes/v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 scale=0.001 0.001 0.001
- link left_inner_knuckle: geometry collision mesh filename=file://$(find robotiq_2f_85_gripper_visualization)/meshes/c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 scale=0.001 0.001 0.001; visual mesh filename=file://$(find robotiq_2f_85_gripper_visualization)/meshes/v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 scale=0.001 0.001 0.001
- link left_outer_finger: geometry collision mesh filename=file://$(find robotiq_2f_85_gripper_visualization)/meshes/c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 scale=0.001 0.001 0.001; visual mesh filename=file://$(find robotiq_2f_85_gripper_visualization)/meshes/v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 scale=0.001 0.001 0.001
- link left_outer_knuckle: geometry collision mesh filename=file://$(find robotiq_2f_85_gripper_visualization)/meshes/c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 scale=0.001 0.001 0.001; visual mesh filename=file://$(find robotiq_2f_85_gripper_visualization)/meshes/v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 scale=0.001 0.001 0.001
- link right_inner_finger: geometry collision mesh filename=file://$(find robotiq_2f_85_gripper_visualization)/meshes/c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 scale=0.001 0.001 0.001; visual mesh filename=file://$(find robotiq_2f_85_gripper_visualization)/meshes/v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 scale=0.001 0.001 0.001
- link right_inner_knuckle: geometry collision mesh filename=file://$(find robotiq_2f_85_gripper_visualization)/meshes/c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 scale=0.001 0.001 0.001; visual mesh filename=file://$(find robotiq_2f_85_gripper_visualization)/meshes/v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 scale=0.001 0.001 0.001
- link right_outer_finger: geometry collision mesh filename=file://$(find robotiq_2f_85_gripper_visualization)/meshes/c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 scale=0.001 0.001 0.001; visual mesh filename=file://$(find robotiq_2f_85_gripper_visualization)/meshes/v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 scale=0.001 0.001 0.001
- link right_outer_knuckle: geometry collision mesh filename=file://$(find robotiq_2f_85_gripper_visualization)/meshes/c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 scale=0.001 0.001 0.001; visual mesh filename=file://$(find robotiq_2f_85_gripper_visualization)/meshes/v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 scale=0.001 0.001 0.001
- link robotiq_arg2f_base_link: geometry collision mesh filename=file://$(find robotiq_2f_85_gripper_visualization)/meshes/c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; visual mesh filename=file://$(find robotiq_2f_85_gripper_visualization)/meshes/v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
