Commit message: Fix urdfs and meshes for mimic joint support.

File: robotiq_2f_85_gripper_visualization/urdf/robotiq_arg2f.xacro (robot description, xacro)
@@ -11,5 +11,5 @@
         <origin xyz="0 0 0" rpy="0 0 0" />
         <geometry>
-          <mesh filename="package://robotiq_2f_85_gripper_visualization/meshes/visual/robotiq_arg2f_85_base_link.dae" scale="0.001 0.001 0.001"/>
+          <mesh filename="package://robotiq_2f_85_gripper_visualization/meshes/visual/robotiq_arg2f_85_base_link.dae" />
         </geometry>
         <material name="">

File: robotiq_2f_85_gripper_visualization/urdf/robotiq_arg2f_85_model_macro.xacro (robot description, xacro)
@@ -136,5 +136,5 @@
       <axis xyz="1 0 0" />
       <limit lower="0" upper="0.8757" velocity="2.0" effort="1000" />
-      <dynamics damping="0.5" />
+      <dynamics damping="3.0" />
       <mimic joint="${prefix}finger_joint" multiplier="1" offset="0" />
     </joint>
@@ -147,5 +147,5 @@
       <axis xyz="1 0 0" />
       <limit lower="-0.8757" upper="0.0" velocity="2.0" effort="1000" />
-      <dynamics damping="0.5" />
+      <dynamics damping="3.0" />
       <mimic joint="${prefix}finger_joint" multiplier="-1" offset="0" />
     </joint>
@@ -167,5 +167,5 @@
       <axis xyz="1 0 0" />
       <limit lower="0" upper="0.8" velocity="2.0" effort="1000" />
-      <dynamics damping="0.5" />
+      <dynamics damping="3.0" />
     </joint>
     <xacro:finger_joints prefix="${prefix}" fingerprefix="left" reflect="1.0"/>
@@ -178,5 +178,5 @@
       <axis xyz="1 0 0" />
       <limit lower="0" upper="0.81" velocity="2.0" effort="1000" />
-      <dynamics damping="0.5" />
+      <dynamics damping="3.0" />
       <mimic joint="${prefix}finger_joint" multiplier="1" offset="0" />
     </joint>

File: robotiq_2f_85_gripper_visualization/urdf/robotiq_gripper.ros2_control.xacro (robot description, xacro)
@@ -22,19 +22,21 @@
                         <param name="initial_value">0.0</param>
                     </state_interface>
-                    <param name="p_pos">10.0</param>
+                    <!-- needed for gripper controller max effort -->
+                    <state_interface name="effort" />
+                    <param name="p_pos">20.0</param>
                     <param name="i_pos">0.0</param>
-                    <param name="d_pos">0.0</param>
-                    <param name="iMax_pos">0.25</param>
-                    <param name="iMin_pos">-0.25</param>
-                    <param name="cmdMax_pos">0.5</param>
-                    <param name="cmdMin_pos">-0.5</param>
+                    <param name="d_pos">0.01</param>
+                    <param name="iMax_pos">0.0</param>
+                    <param name="iMin_pos">0.0</param>
+                    <param name="cmdMax_pos">2.0</param>
+                    <param name="cmdMin_pos">-2.0</param>
                     <param name="cmdOffset_pos">0.0</param>
-                    <param name="p_vel">100.0</param>
-                    <param name="i_vel">100.0</param>
+                    <param name="p_vel">2.5</param>
+                    <param name="i_vel">0.1</param>
                     <param name="d_vel">0.0</param>
-                    <param name="iMax_vel">0.0</param>
-                    <param name="iMin_vel">-0.0</param>
-                    <param name="cmdMax_vel">50.0</param>
-                    <param name="cmdMin_vel">-50.0</param>
+                    <param name="iMax_vel">1.0</param>
+                    <param name="iMin_vel">-1.0</param>
+                    <param name="cmdMax_vel">1000.0</param>
+                    <param name="cmdMin_vel">-1000.0</param>
                     <param name="cmdOffset_vel">0.0</param>
                 </xacro:if>
@@ -45,139 +47,4 @@
                 <command_interface name="position" />
                 <state_interface name="velocity"/>
-            </joint>
-            <joint name="${prefix}right_outer_knuckle_joint">
-                <param name="mimic">${prefix}finger_joint</param>
-                <param name="multiplier">1</param>
-                <xacro:unless value="${sim_ignition}">
-                    <command_interface name="position"/>
-                    <state_interface name="position"/>
-                    <state_interface name="velocity"/>
-                </xacro:unless>
-                <xacro:if value="${sim_ignition}">
-                  <param name="p_pos">100.0</param>
-                  <param name="i_pos">0.0</param>
-                  <param name="d_pos">0.0</param>
-                  <param name="iMax_pos">0.25</param>
-                  <param name="iMin_pos">-0.25</param>
-                  <param name="cmdMax_pos">0.5</param>
-                  <param name="cmdMin_pos">-0.5</param>
-                  <param name="cmdOffset_pos">0.0</param>
-                  <param name="p_vel">100.0</param>
-                  <param name="i_vel">1.0</param>
-                  <param name="d_vel">0.0</param>
-                  <param name="iMax_vel">25.0</param>
-                  <param name="iMin_vel">-25.0</param>
-                  <param name="cmdMax_vel">50.0</param>
-                  <param name="cmdMin_vel">-50.0</param>
-                  <param name="cmdOffset_vel">0.0</param>
-                </xacro:if>
-            </joint>
-            <joint name="${prefix}left_inner_knuckle_joint">
-                <param name="mimic">${prefix}finger_joint</param>
-                <param name="multiplier">1</param>
-                <xacro:unless value="${sim_ignition}">
-                    <command_interface name="position"/>
-                    <state_interface name="position"/>
-                    <state_interface name="velocity"/>
-                </xacro:unless>
-                <xacro:if value="${sim_ignition}">
-                  <param name="p_pos">100.0</param>
-                  <param name="i_pos">0.0</param>
-                  <param name="d_pos">0.0</param>
-                  <param name="iMax_pos">0.25</param>
-                  <param name="iMin_pos">-0.25</param>
-                  <param name="cmdMax_pos">0.5</param>
-                  <param name="cmdMin_pos">-0.5</param>
-                  <param name="cmdOffset_pos">0.0</param>
-                  <param name="p_vel">100.0</param>
-                  <param name="i_vel">1.0</param>
-                  <param name="d_vel">0.0</param>
-                  <param name="iMax_vel">0.0</param>
-                  <param name="iMin_vel">-0.0</param>
-                  <param name="cmdMax_vel">50.0</param>
-                  <param name="cmdMin_vel">-50.0</param>
-                  <param name="cmdOffset_vel">0.0</param>
-                </xacro:if>
-            </joint>
-            <joint name="${prefix}right_inner_knuckle_joint">
-                <param name="mimic">${prefix}finger_joint</param>
-                <param name="multiplier">1</param>
-                <xacro:unless value="${sim_ignition}">
-                    <command_interface name="position"/>
-                    <state_interface name="position"/>
-                    <state_interface name="velocity"/>
-                </xacro:unless>
-                <xacro:if value="${sim_ignition}">
-                  <param name="p_pos">100.0</param>
-                  <param name="i_pos">0.0</param>
-                  <param name="d_pos">0.0</param>
-                  <param name="iMax_pos">0.25</param>
-                  <param name="iMin_pos">-0.25</param>
-                  <param name="cmdMax_pos">0.5</param>
-                  <param name="cmdMin_pos">-0.5</param>
-                  <param name="cmdOffset_pos">0.0</param>
-                  <param name="p_vel">100.0</param>
-                  <param name="i_vel">1.0</param>
-                  <param name="d_vel">0.0</param>
-                  <param name="iMax_vel">25.0</param>
-                  <param name="iMin_vel">-25.0</param>
-                  <param name="cmdMax_vel">50.0</param>
-                  <param name="cmdMin_vel">-50.0</param>
-                  <param name="cmdOffset_vel">0.0</param>
-                </xacro:if>
-            </joint>
-            <joint name="${prefix}left_inner_finger_joint">
-                <param name="mimic">${prefix}finger_joint</param>
-                <param name="multiplier">-1</param>
-                <xacro:unless value="${sim_ignition}">
-                    <command_interface name="position"/>
-                    <state_interface name="position"/>
-                    <state_interface name="velocity"/>
-                </xacro:unless>
-                <xacro:if value="${sim_ignition}">
-                  <param name="p_pos">10.0</param>
-                  <param name="i_pos">0.0</param>
-                  <param name="d_pos">0.0</param>
-                  <param name="iMax_pos">0.25</param>
-                  <param name="iMin_pos">-0.25</param>
-                  <param name="cmdMax_pos">0.5</param>
-                  <param name="cmdMin_pos">-0.5</param>
-                  <param name="cmdOffset_pos">0.0</param>
-                  <param name="p_vel">100.0</param>
-                  <param name="i_vel">100.0</param>
-                  <param name="d_vel">0.0</param>
-                  <param name="iMax_vel">0.0</param>
-                  <param name="iMin_vel">-0.0</param>
-                  <param name="cmdMax_vel">50.0</param>
-                  <param name="cmdMin_vel">-50.0</param>
-                  <param name="cmdOffset_vel">0.0</param>
-                </xacro:if>
-            </joint>
-            <joint name="${prefix}right_inner_finger_joint">
-                <param name="mimic">${prefix}finger_joint</param>
-                <param name="multiplier">-1</param>
-                <xacro:unless value="${sim_ignition}">
-                    <command_interface name="position"/>
-                    <state_interface name="position"/>
-                    <state_interface name="velocity"/>
-                </xacro:unless>
-                <xacro:if value="${sim_ignition}">
-                  <param name="p_pos">10.0</param>
-                  <param name="i_pos">0.0</param>
-                  <param name="d_pos">0.0</param>
-                  <param name="iMax_pos">0.25</param>
-                  <param name="iMin_pos">-0.25</param>
-                  <param name="cmdMax_pos">0.5</param>
-                  <param name="cmdMin_pos">-0.5</param>
-                  <param name="cmdOffset_pos">0.0</param>
-                  <param name="p_vel">100.0</param>
-                  <param name="i_vel">100.0</param>
-                  <param name="d_vel">0.0</param>
-                  <param name="iMax_vel">25.0</param>
-                  <param name="iMin_vel">-25.0</param>
-                  <param name="cmdMax_vel">50.0</param>
-                  <param name="cmdMin_vel">-50.0</param>
-                  <param name="cmdOffset_vel">0.0</param>
-                </xacro:if>
             </joint>
             <!-- Only add this with fake hardware mode -->

File: robotiq_2f_85_gripper_visualization/urdf/robotiq_gripper.urdf.xacro (robot description, xacro)
@@ -25,4 +25,108 @@
                 <parameters>$(find robotiq_bringup)/config/robotiq_2f_85_controllers.yaml</parameters>
             </plugin>
+            <plugin filename="mimic-joint-system" name="ign_ros2_control::MimicJointSystem">
+                <joint_name>right_outer_knuckle_joint</joint_name>
+                <mimic_joint_name>finger_joint</mimic_joint_name>
+                <multiplier>1.0</multiplier>
+                <offset>0.0</offset>
+                <joint_index>0</joint_index>
+                <mimic_joint_index>0</mimic_joint_index>
+                <p_gain>100.0</p_gain>
+                <i_gain>0.1</i_gain>
+                <d_gain>0.0</d_gain>
+                <i_max>5.0</i_max>
+                <i_min>-5.0</i_min>
+                <cmd_max>500.0</cmd_max>
+                <cmd_min>-500.0</cmd_min>
+                <cmd_offset>0.0</cmd_offset>
+                <dead_zone>0.001</dead_zone>
+                <use_velocity_commands>false</use_velocity_commands>
+            </plugin>
+            <plugin filename="mimic-joint-system" name="ign_ros2_control::MimicJointSystem">
+                <joint_name>left_inner_knuckle_joint</joint_name>
+                <mimic_joint_name>finger_joint</mimic_joint_name>
+                <multiplier>1.0</multiplier>
+                <offset>0.0</offset>
+                <joint_index>0</joint_index>
+                <mimic_joint_index>0</mimic_joint_index>
+                <p_gain>100.0</p_gain>
+                <i_gain>0.1</i_gain>
+                <d_gain>0.0</d_gain>
+                <i_max>5.0</i_max>
+                <i_min>-5.0</i_min>
+                <cmd_max>500.0</cmd_max>
+                <cmd_min>-500.0</cmd_min>
+                <cmd_offset>0.0</cmd_offset>
+                <dead_zone>0.001</dead_zone>
+                <use_velocity_commands>false</use_velocity_commands>
+            </plugin>
+            <plugin filename="mimic-joint-system" name="ign_ros2_control::MimicJointSystem">
+                <joint_name>right_inner_knuckle_joint</joint_name>
+                <mimic_joint_name>finger_joint</mimic_joint_name>
+                <multiplier>1.0</multiplier>
+                <offset>0.0</offset>
+                <joint_index>0</joint_index>
+                <mimic_joint_index>0</mimic_joint_index>
+                <p_gain>100.0</p_gain>
+                <i_gain>0.1</i_gain>
+                <d_gain>0.0</d_gain>
+                <i_max>5.0</i_max>
+                <i_min>-5.0</i_min>
+                <cmd_max>500.0</cmd_max>
+                <cmd_min>-500.0</cmd_min>
+                <cmd_offset>0.0</cmd_offset>
+                <dead_zone>0.001</dead_zone>
+                <use_velocity_commands>false</use_velocity_commands>
+            </plugin>
+            <plugin filename="mimic-joint-system" name="ign_ros2_control::MimicJointSystem">
+                <joint_name>left_inner_finger_joint</joint_name>
+                <mimic_joint_name>finger_joint</mimic_joint_name>
+                <multiplier>-1.0</multiplier>
+                <offset>0.0</offset>
+                <joint_index>0</joint_index>
+                <mimic_joint_index>0</mimic_joint_index>
+                <p_gain>100.0</p_gain>
+                <i_gain>0.1</i_gain>
+                <d_gain>0.0</d_gain>
+                <i_max>1.0</i_max>
+                <i_min>-1.0</i_min>
+                <cmd_max>500.0</cmd_max>
+                <cmd_min>-500.0</cmd_min>
+                <cmd_offset>0.0</cmd_offset>
+                <dead_zone>0.001</dead_zone>
+                <use_velocity_commands>false</use_velocity_commands>
+            </plugin>
+            <plugin filename="mimic-joint-system" name="ign_ros2_control::MimicJointSystem">
+                <joint_name>right_inner_finger_joint</joint_name>
+                <mimic_joint_name>finger_joint</mimic_joint_name>
+                <multiplier>-1.0</multiplier>
+                <offset>0.0</offset>
+                <joint_index>0</joint_index>
+                <mimic_joint_index>0</mimic_joint_index>
+                <p_gain>100.0</p_gain>
+                <i_gain>0.1</i_gain>
+                <d_gain>0.0</d_gain>
+                <i_max>5.0</i_max>
+                <i_min>-5.0</i_min>
+                <cmd_max>500.0</cmd_max>
+                <cmd_min>-500.0</cmd_min>
+                <cmd_offset>0.0</cmd_offset>
+                <dead_zone>0.001</dead_zone>
+                <use_velocity_commands>false</use_velocity_commands>
+            </plugin>
+            <!-- for test -->
+<!--            <plugin-->
+<!--                    filename="ignition-gazebo-joint-position-controller-system"-->
+<!--                    name="ignition::gazebo::systems::JointPositionController">-->
+<!--                <joint_name>finger_joint</joint_name>-->
+<!--                <topic>rotor_cmd</topic>-->
+<!--                <p_gain>50.0</p_gain>-->
+<!--                <i_gain>0.1</i_gain>-->
+<!--                <d_gain>0.0</d_gain>-->
+<!--                <i_max>1</i_max>-->
+<!--                <i_min>-1</i_min>-->
+<!--                <cmd_max>1000</cmd_max>-->
+<!--                <cmd_min>-1000</cmd_min>-->
+<!--            </plugin>-->
         </gazebo>
     </xacro:if>
