Commit message: Add absolute path option.

File: robotiq_2f_85_gripper_visualization/urdf/robotiq_arg2f.xacro (robot description, xacro)
@@ -1,5 +1,5 @@
 <?xml version="1.0"?>
 <robot xmlns:xacro="http://ros.org/wiki/xacro">
-  <xacro:macro name="robotiq_arg2f_base_link" params="prefix">
+  <xacro:macro name="robotiq_arg2f_base_link" params="prefix force_abs_paths:=false">
     <link name="${prefix}robotiq_arg2f_base_link">
       <inertial>
@@ -11,5 +11,10 @@
         <origin xyz="0 0 0" rpy="0 0 0" />
         <geometry>
-          <mesh filename="package://robotiq_2f_85_gripper_visualization/meshes/visual/robotiq_arg2f_85_base_link.dae" />
+          <xacro:if value="${force_abs_paths}">
+            <mesh filename="file://$(find robotiq_2f_85_gripper_visualization)/meshes/visual/robotiq_arg2f_85_base_link.dae" />
+          </xacro:if>
+          <xacro:unless value="${force_abs_paths}">
+            <mesh filename="package://robotiq_2f_85_gripper_visualization/meshes/visual/robotiq_arg2f_85_base_link.dae" />
+          </xacro:unless>
         </geometry>
         <material name="">
@@ -20,5 +25,10 @@
         <origin xyz="0 0 0" rpy="0 0 0" />
         <geometry>
-           <mesh filename="package://robotiq_2f_85_gripper_visualization/meshes/collision/robotiq_arg2f_base_link.stl" />
+          <xacro:if value="${force_abs_paths}">
+            <mesh filename="file://$(find robotiq_2f_85_gripper_visualization)/meshes/collision/robotiq_arg2f_base_link.stl" />
+          </xacro:if>
+          <xacro:unless value="${force_abs_paths}">
+            <mesh filename="package://robotiq_2f_85_gripper_visualization/meshes/collision/robotiq_arg2f_base_link.stl" />
+          </xacro:unless>
         </geometry>
       </collision>
@@ -31,10 +41,10 @@
     <xacro:inner_finger_pad_joint prefix="${prefix}" fingerprefix="${fingerprefix}"/>
   </xacro:macro>
-  <xacro:macro name="finger_links" params="prefix fingerprefix stroke">
-    <xacro:outer_knuckle prefix="${prefix}" fingerprefix="${fingerprefix}" stroke="${stroke}"/>
-    <xacro:outer_finger prefix="${prefix}" fingerprefix="${fingerprefix}" stroke="${stroke}"/>
-    <xacro:inner_finger prefix="${prefix}" fingerprefix="${fingerprefix}" stroke="${stroke}"/>
-    <xacro:inner_finger_pad prefix="${prefix}" fingerprefix="${fingerprefix}"/>
-    <xacro:inner_knuckle prefix="${prefix}" fingerprefix="${fingerprefix}" stroke="${stroke}"/>
+  <xacro:macro name="finger_links" params="prefix fingerprefix stroke force_abs_paths:=false">
+    <xacro:outer_knuckle prefix="${prefix}" fingerprefix="${fingerprefix}" stroke="${stroke}" force_abs_paths="${force_abs_paths}"/>
+    <xacro:outer_finger prefix="${prefix}" fingerprefix="${fingerprefix}" stroke="${stroke}" force_abs_paths="${force_abs_paths}"/>
+    <xacro:inner_finger prefix="${prefix}" fingerprefix="${fingerprefix}" stroke="${stroke}" force_abs_paths="${force_abs_paths}"/>
+    <xacro:inner_finger_pad prefix="${prefix}" fingerprefix="${fingerprefix}" force_abs_paths="${force_abs_paths}"/>
+    <xacro:inner_knuckle prefix="${prefix}" fingerprefix="${fingerprefix}" stroke="${stroke}" force_abs_paths="${force_abs_paths}"/>
   </xacro:macro>
 </robot>

File: robotiq_2f_85_gripper_visualization/urdf/robotiq_arg2f_85_model_macro.xacro (robot description, xacro)
@@ -1,5 +1,5 @@
 <?xml version="1.0"?>
 <robot xmlns:xacro="http://ros.org/wiki/xacro">
-  <xacro:macro name="outer_knuckle" params="prefix fingerprefix stroke">
+  <xacro:macro name="outer_knuckle" params="prefix fingerprefix stroke force_abs_paths:=false">
     <link name="${prefix}${fingerprefix}_outer_knuckle">
       <inertial>
@@ -11,5 +11,10 @@
         <origin xyz="0 0 0" rpy="0 0 0" />
         <geometry>
-          <mesh filename="package://robotiq_2f_85_gripper_visualization/meshes/visual/robotiq_arg2f_85_outer_knuckle.dae" scale="0.001 0.001 0.001"/>
+          <xacro:if value="${force_abs_paths}">
+            <mesh filename="file://$(find robotiq_2f_85_gripper_visualization)/meshes/visual/robotiq_arg2f_85_outer_knuckle.dae" scale="0.001 0.001 0.001"/>
+          </xacro:if>
+          <xacro:unless value="${force_abs_paths}">
+            <mesh filename="package://robotiq_2f_85_gripper_visualization/meshes/visual/robotiq_arg2f_85_outer_knuckle.dae" scale="0.001 0.001 0.001"/>
+          </xacro:unless>
         </geometry>
         <material name="">
@@ -20,10 +25,15 @@
         <origin xyz="0 0 0" rpy="0 0 0" />
         <geometry>
-          <mesh filename="package://robotiq_2f_85_gripper_visualization/meshes/collision/robotiq_arg2f_85_outer_knuckle.dae" scale="0.001 0.001 0.001"/>
-        </geometry>
-      </collision>
-    </link>
-  </xacro:macro>
-  <xacro:macro name="outer_finger" params="prefix fingerprefix stroke">
+          <xacro:if value="${force_abs_paths}">
+            <mesh filename="file://$(find robotiq_2f_85_gripper_visualization)/meshes/collision/robotiq_arg2f_85_outer_knuckle.dae" scale="0.001 0.001 0.001"/>
+          </xacro:if>
+          <xacro:unless value="${force_abs_paths}">
+            <mesh filename="package://robotiq_2f_85_gripper_visualization/meshes/collision/robotiq_arg2f_85_outer_knuckle.dae" scale="0.001 0.001 0.001"/>
+          </xacro:unless>
+        </geometry>
+      </collision>
+    </link>
+  </xacro:macro>
+  <xacro:macro name="outer_finger" params="prefix fingerprefix stroke force_abs_paths:=false">
     <link name="${prefix}${fingerprefix}_outer_finger">
       <inertial>
@@ -35,5 +45,10 @@
         <origin xyz="0 0 0" rpy="0 0 0" />
         <geometry>
-          <mesh filename="package://robotiq_2f_85_gripper_visualization/meshes/visual/robotiq_arg2f_85_outer_finger.dae" scale="0.001 0.001 0.001"/>
+          <xacro:if value="${force_abs_paths}">
+            <mesh filename="file://$(find robotiq_2f_85_gripper_visualization)/meshes/visual/robotiq_arg2f_85_outer_finger.dae" scale="0.001 0.001 0.001"/>
+          </xacro:if>
+          <xacro:unless value="${force_abs_paths}">
+            <mesh filename="package://robotiq_2f_85_gripper_visualization/meshes/visual/robotiq_arg2f_85_outer_finger.dae" scale="0.001 0.001 0.001"/>
+          </xacro:unless>
         </geometry>
         <material name="">
@@ -44,10 +59,15 @@
         <origin xyz="0 0 0" rpy="0 0 0" />
         <geometry>
-          <mesh filename="package://robotiq_2f_85_gripper_visualization/meshes/collision/robotiq_arg2f_85_outer_finger.dae" scale="0.001 0.001 0.001"/>
-        </geometry>
-      </collision>
-    </link>
-  </xacro:macro>
-  <xacro:macro name="inner_knuckle" params="prefix fingerprefix stroke">
+          <xacro:if value="${force_abs_paths}">
+            <mesh filename="file://$(find robotiq_2f_85_gripper_visualization)/meshes/collision/robotiq_arg2f_85_outer_finger.dae" scale="0.001 0.001 0.001"/>
+          </xacro:if>
+          <xacro:unless value="${force_abs_paths}">
+            <mesh filename="package://robotiq_2f_85_gripper_visualization/meshes/collision/robotiq_arg2f_85_outer_finger.dae" scale="0.001 0.001 0.001"/>
+          </xacro:unless>
+        </geometry>
+      </collision>
+    </link>
+  </xacro:macro>
+  <xacro:macro name="inner_knuckle" params="prefix fingerprefix stroke force_abs_paths:=false">
     <link name="${prefix}${fingerprefix}_inner_knuckle">
       <inertial>
@@ -59,5 +79,10 @@
         <origin xyz="0 0 0" rpy="0 0 0" />
         <geometry>
-          <mesh filename="package://robotiq_2f_85_gripper_visualization/meshes/visual/robotiq_arg2f_85_inner_knuckle.dae" scale="0.001 0.001 0.001"/>
+          <xacro:if value="${force_abs_paths}">
+            <mesh filename="file://$(find robotiq_2f_85_gripper_visualization)/meshes/visual/robotiq_arg2f_85_inner_knuckle.dae" scale="0.001 0.001 0.001"/>
+          </xacro:if>
+          <xacro:unless value="${force_abs_paths}">
+            <mesh filename="package://robotiq_2f_85_gripper_visualization/meshes/visual/robotiq_arg2f_85_inner_knuckle.dae" scale="0.001 0.001 0.001"/>
+          </xacro:unless>
         </geometry>
         <material name="">
@@ -68,10 +93,15 @@
         <origin xyz="0 0 0" rpy="0 0 0" />
         <geometry>
-          <mesh filename="package://robotiq_2f_85_gripper_visualization/meshes/collision/robotiq_arg2f_85_inner_knuckle.dae" scale="0.001 0.001 0.001"/>
-        </geometry>
-      </collision>
-    </link>
-  </xacro:macro>
-  <xacro:macro name="inner_finger" params="prefix fingerprefix stroke">
+          <xacro:if value="${force_abs_paths}">
+            <mesh filename="file://$(find robotiq_2f_85_gripper_visualization)/meshes/collision/robotiq_arg2f_85_inner_knuckle.dae" scale="0.001 0.001 0.001"/>
+          </xacro:if>
+          <xacro:unless value="${force_abs_paths}">
+            <mesh filename="package://robotiq_2f_85_gripper_visualization/meshes/collision/robotiq_arg2f_85_inner_knuckle.dae" scale="0.001 0.001 0.001"/>
+          </xacro:unless>
+        </geometry>
+      </collision>
+    </link>
+  </xacro:macro>
+  <xacro:macro name="inner_finger" params="prefix fingerprefix stroke force_abs_paths:=false">
     <link name="${prefix}${fingerprefix}_inner_finger">
       <inertial>
@@ -83,5 +113,10 @@
         <origin xyz="0 0 0" rpy="0 0 0" />
         <geometry>
-          <mesh filename="package://robotiq_2f_85_gripper_visualization/meshes/visual/robotiq_arg2f_85_inner_finger.dae" scale="0.001 0.001 0.001"/>
+          <xacro:if value="${force_abs_paths}">
+            <mesh filename="file://$(find robotiq_2f_85_gripper_visualization)/meshes/visual/robotiq_arg2f_85_inner_finger.dae" scale="0.001 0.001 0.001"/>
+          </xacro:if>
+          <xacro:unless value="${force_abs_paths}">
+            <mesh filename="package://robotiq_2f_85_gripper_visualization/meshes/visual/robotiq_arg2f_85_inner_finger.dae" scale="0.001 0.001 0.001"/>
+          </xacro:unless>
         </geometry>
         <material name="">
@@ -92,5 +127,10 @@
         <origin xyz="0 0 0" rpy="0 0 0" />
         <geometry>
-          <mesh filename="package://robotiq_2f_85_gripper_visualization/meshes/collision/robotiq_arg2f_85_inner_finger.dae" scale="0.001 0.001 0.001" />
+          <xacro:if value="${force_abs_paths}">
+            <mesh filename="file://$(find robotiq_2f_85_gripper_visualization)/meshes/collision/robotiq_arg2f_85_inner_finger.dae" scale="0.001 0.001 0.001"/>
+          </xacro:if>
+          <xacro:unless value="${force_abs_paths}">
+            <mesh filename="package://robotiq_2f_85_gripper_visualization/meshes/collision/robotiq_arg2f_85_inner_finger.dae" scale="0.001 0.001 0.001" />
+          </xacro:unless>
         </geometry>
       </collision>
@@ -98,5 +138,5 @@
   </xacro:macro>
    <!-- Finger pad link, the default are the "big pads" with rubber-->
-  <xacro:macro name="inner_finger_pad" params="prefix fingerprefix">
+  <xacro:macro name="inner_finger_pad" params="prefix fingerprefix force_abs_paths:=false">
     <link name="${prefix}${fingerprefix}_inner_finger_pad">
       <visual>
@@ -184,8 +224,8 @@
   </xacro:macro>
   <!-- Initialization of all joints and links -->
-  <xacro:macro name="robotiq_arg2f_85" params="prefix">
-    <xacro:robotiq_arg2f_base_link prefix="${prefix}"/>
-    <xacro:finger_links prefix="${prefix}" fingerprefix="left" stroke="85"/>
-    <xacro:finger_links prefix="${prefix}" fingerprefix="right" stroke="85"/>
+  <xacro:macro name="robotiq_arg2f_85" params="prefix force_abs_paths:=false">
+    <xacro:robotiq_arg2f_base_link prefix="${prefix}" force_abs_paths="${force_abs_paths}"/>
+    <xacro:finger_links prefix="${prefix}" fingerprefix="left" stroke="85" force_abs_paths="${force_abs_paths}"/>
+    <xacro:finger_links prefix="${prefix}" fingerprefix="right" stroke="85" force_abs_paths="${force_abs_paths}"/>
     <xacro:finger_joint prefix="${prefix}"/>
     <xacro:right_outer_knuckle_joint prefix="${prefix}"/>

File: robotiq_2f_85_gripper_visualization/urdf/robotiq_gripper.urdf.xacro (robot description, xacro)
@@ -5,4 +5,5 @@
     <xacro:arg name="prefix" default="" />
     <xacro:arg name="sim_ignition" default="false" />
+    <xacro:arg name="force_abs_path" default="false" />
     <!-- Import macros -->
     <xacro:include filename="$(find robotiq_2f_85_gripper_visualization)/urdf/robotiq_arg2f_85_model_macro.xacro" />
@@ -14,5 +15,5 @@
         <child link="$(arg prefix)robotiq_arg2f_base_link"/>
     </joint>
-    <xacro:robotiq_arg2f_85 prefix="$(arg prefix)"/>
+    <xacro:robotiq_arg2f_85 prefix="$(arg prefix)" force_abs_paths="$(arg force_abs_paths)"/>
     <xacro:robotiq_sim_gripper_ros2_control name="RobotiqGripperSystem"
                                             prefix="$(arg prefix)"

File: robotiq_2f_85_gripper_visualization/urdf/robotiq_gripper_macro.urdf.xacro (robot description, xacro)
@@ -8,5 +8,6 @@
         sim_ignition:=false
         use_fake_hardware:=false
-        fake_sensor_commands:=false">
+        fake_sensor_commands:=false
+        force_abs_paths:=false" >
     <!-- Import macros -->
     <xacro:include filename="$(find robotiq_2f_85_gripper_visualization)/urdf/robotiq_arg2f_85_model_macro.xacro" />
@@ -17,5 +18,5 @@
       <xacro:insert_block name="origin" />
     </joint>
-    <xacro:robotiq_arg2f_85 prefix="$(arg prefix)"/>
+    <xacro:robotiq_arg2f_85 prefix="$(arg prefix)" force_abs_paths="${force_abs_paths}"/>
     <xacro:robotiq_sim_gripper_ros2_control name="RobotiqGripperSystem"
                                             prefix="${prefix}"
