Commit message: Add full macro. Friciton coeffs.

File: robotiq_2f_85_gripper_visualization/urdf/robotiq_gripper.ros2_control.xacro (robot description, xacro)
@@ -16,35 +16,143 @@
             </hardware>
             <!-- Joint interfaces -->
-            <joint name="${prefix}finger_joint">
-                <!-- With Ignition, we have mimic joints, so we only need this command interface activated -->
-                <xacro:if value="${sim_ignition}">
-                    <state_interface name="position">
-                        <param name="initial_value">0.0</param>
-                    </state_interface>
-                    <!-- needed for gripper controller max effort -->
-                    <state_interface name="effort" />
-                    <param name="p_pos">20.0</param>
-                    <param name="i_pos">0.0</param>
-                    <param name="d_pos">0.01</param>
-                    <param name="iMax_pos">0.0</param>
-                    <param name="iMin_pos">0.0</param>
-                    <param name="cmdMax_pos">2.0</param>
-                    <param name="cmdMin_pos">-2.0</param>
-                    <param name="cmdOffset_pos">0.0</param>
-                    <param name="p_vel">2.5</param>
-                    <param name="i_vel">0.1</param>
-                    <param name="d_vel">0.0</param>
-                    <param name="iMax_vel">1.0</param>
-                    <param name="iMin_vel">-1.0</param>
-                    <param name="cmdMax_vel">1000.0</param>
-                    <param name="cmdMin_vel">-1000.0</param>
-                    <param name="cmdOffset_vel">0.0</param>
-                </xacro:if>
-                <xacro:unless value="${sim_ignition}">
-                    <param name="initial_position">0.0</param>
-                    <state_interface name="position"/>
-                </xacro:unless>
-                <command_interface name="position" />
+            <joint name="finger_joint">
+                <state_interface name="position">
+                    <param name="initial_value">0.0</param>
+                </state_interface>
+                <!-- needed for gripper controller max effort -->
+                <state_interface name="effort"/>
+                <param name="p_pos">20.0</param>
+                <param name="i_pos">0.0</param>
+                <param name="d_pos">0.01</param>
+                <param name="iMax_pos">0.0</param>
+                <param name="iMin_pos">0.0</param>
+                <param name="cmdMax_pos">2.0</param>
+                <param name="cmdMin_pos">-2.0</param>
+                <param name="cmdOffset_pos">0.0</param>
+                <param name="p_vel">100.0</param>
+                <param name="i_vel">1.0</param>
+                <param name="d_vel">0.0</param>
+                <param name="iMax_vel">1.0</param>
+                <param name="iMin_vel">-1.0</param>
+                <param name="cmdMax_vel">1000.0</param>
+                <param name="cmdMin_vel">-1000.0</param>
+                <param name="cmdOffset_vel">0.0</param>
+                <command_interface name="position"/>
                 <state_interface name="velocity"/>
+            </joint>
+            <joint name="right_outer_knuckle_joint">
+                <param name="mimic">finger_joint</param>
+                <param name="multiplier">1</param>
+                <state_interface name="position"/>
+                <param name="p_pos">20.0</param>
+                <param name="i_pos">0.0</param>
+                <param name="d_pos">0.01</param>
+                <param name="iMax_pos">0.0</param>
+                <param name="iMin_pos">0.0</param>
+                <param name="cmdMax_pos">2.0</param>
+                <param name="cmdMin_pos">-2.0</param>
+                <param name="cmdOffset_pos">0.0</param>
+                <param name="p_vel">100.0</param>
+                <param name="i_vel">1.0</param>
+                <param name="d_vel">0.0</param>
+                <param name="iMax_vel">50.0</param>
+                <param name="iMin_vel">-50.0</param>
+                <param name="cmdMax_vel">1000.0</param>
+                <param name="cmdMin_vel">-1000.0</param>
+                <param name="cmdOffset_vel">0.0</param>
+                <state_interface name="velocity"/>
+                <state_interface name="effort"/>
+            </joint>
+            <joint name="left_inner_knuckle_joint">
+                <param name="mimic">finger_joint</param>
+                <param name="multiplier">1</param>
+                <state_interface name="position"/>
+                <param name="p_pos">20.0</param>
+                <param name="i_pos">0.0</param>
+                <param name="d_pos">0.01</param>
+                <param name="iMax_pos">0.0</param>
+                <param name="iMin_pos">0.0</param>
+                <param name="cmdMax_pos">2.0</param>
+                <param name="cmdMin_pos">-2.0</param>
+                <param name="cmdOffset_pos">0.0</param>
+                <param name="p_vel">100.0</param>
+                <param name="i_vel">1.0</param>
+                <param name="d_vel">0.0</param>
+                <param name="iMax_vel">50.0</param>
+                <param name="iMin_vel">-50.0</param>
+                <param name="cmdMax_vel">1000.0</param>
+                <param name="cmdMin_vel">-1000.0</param>
+                <param name="cmdOffset_vel">0.0</param>
+                <state_interface name="velocity"/>
+                <state_interface name="effort"/>
+            </joint>
+            <joint name="right_inner_knuckle_joint">
+                <param name="mimic">finger_joint</param>
+                <param name="multiplier">1</param>
+                <state_interface name="position"/>
+                <param name="p_pos">20.0</param>
+                <param name="i_pos">0.0</param>
+                <param name="d_pos">0.01</param>
+                <param name="iMax_pos">0.0</param>
+                <param name="iMin_pos">0.0</param>
+                <param name="cmdMax_pos">2.0</param>
+                <param name="cmdMin_pos">-2.0</param>
+                <param name="cmdOffset_pos">0.0</param>
+                <param name="p_vel">100.0</param>
+                <param name="i_vel">1.0</param>
+                <param name="d_vel">0.0</param>
+                <param name="iMax_vel">50.0</param>
+                <param name="iMin_vel">-50.0</param>
+                <param name="cmdMax_vel">1000.0</param>
+                <param name="cmdMin_vel">-1000.0</param>
+                <param name="cmdOffset_vel">0.0</param>
+                <state_interface name="velocity"/>
+                <state_interface name="effort"/>
+            </joint>
+            <joint name="left_inner_finger_joint">
+                <param name="mimic">finger_joint</param>
+                <param name="multiplier">-1</param>
+                <state_interface name="position"/>
+                <param name="p_pos">20.0</param>
+                <param name="i_pos">0.0</param>
+                <param name="d_pos">0.01</param>
+                <param name="iMax_pos">0.0</param>
+                <param name="iMin_pos">0.0</param>
+                <param name="cmdMax_pos">2.0</param>
+                <param name="cmdMin_pos">-2.0</param>
+                <param name="cmdOffset_pos">0.0</param>
+                <param name="p_vel">200.0</param>
+                <param name="i_vel">1.0</param>
+                <param name="d_vel">0.0</param>
+                <param name="iMax_vel">1.0</param>
+                <param name="iMin_vel">-1.0</param>
+                <param name="cmdMax_vel">1000.0</param>
+                <param name="cmdMin_vel">-1000.0</param>
+                <param name="cmdOffset_vel">0.0</param>
+                <state_interface name="velocity"/>
+                <state_interface name="effort"/>
+            </joint>
+            <joint name="right_inner_finger_joint">
+                <param name="mimic">finger_joint</param>
+                <param name="multiplier">-1</param>
+                <state_interface name="position"/>
+                <param name="p_pos">20.0</param>
+                <param name="i_pos">0.0</param>
+                <param name="d_pos">0.01</param>
+                <param name="iMax_pos">0.0</param>
+                <param name="iMin_pos">0.0</param>
+                <param name="cmdMax_pos">2.0</param>
+                <param name="cmdMin_pos">-2.0</param>
+                <param name="cmdOffset_pos">0.0</param>
+                <param name="p_vel">200.0</param>
+                <param name="i_vel">1.0</param>
+                <param name="d_vel">0.0</param>
+                <param name="iMax_vel">1.0</param>
+                <param name="iMin_vel">-1.0</param>
+                <param name="cmdMax_vel">1000.0</param>
+                <param name="cmdMin_vel">-1000.0</param>
+                <param name="cmdOffset_vel">0.0</param>
+                <state_interface name="velocity"/>
+                <state_interface name="effort"/>
             </joint>
             <!-- Only add this with fake hardware mode -->

Commit message: Adapt pid values for finger joint.

File: robotiq_2f_85_gripper_visualization/urdf/robotiq_gripper.ros2_control.xacro (robot description, xacro)
@@ -30,5 +30,5 @@
                 <param name="cmdMin_pos">-2.0</param>
                 <param name="cmdOffset_pos">0.0</param>
-                <param name="p_vel">100.0</param>
+                <param name="p_vel">500.0</param>
                 <param name="i_vel">1.0</param>
                 <param name="d_vel">0.0</param>

File: robotiq_2f_85_gripper_visualization/urdf/robotiq_gripper.urdf (robot description, URDF)
Before this commit: robot robotiq_gripper, 13 links, 12 joints
Joints:
- joint finger_joint: limit lower=0 upper=0.8 effort=50 velocity=0.5 -> lower=0 upper=0.8 effort=1000 velocity=2.0
- joint left_inner_finger_joint: limit lower=-0.8757 upper=0.0 effort=50 velocity=0.5 -> lower=-0.8 upper=0.0 effort=1000 velocity=2.0
- joint left_inner_knuckle_joint: limit lower=0 upper=0.8757 effort=50 velocity=0.5 -> lower=0 upper=0.8 effort=1000 velocity=2.0
- joint right_inner_finger_joint: limit lower=-0.8757 upper=0.0 effort=50 velocity=0.5 -> lower=-0.8 upper=0.0 effort=1000 velocity=2.0
- joint right_inner_knuckle_joint: limit lower=0 upper=0.8757 effort=50 velocity=0.5 -> lower=0 upper=0.8 effort=1000 velocity=2.0
- joint right_outer_knuckle_joint: limit lower=0 upper=0.81 effort=50 velocity=0.5 -> lower=0 upper=0.8 effort=1000 velocity=2.0
