Commit message: Improve fake hw launch files and urdfs.

File: robotiq_2f_85_gripper_visualization/urdf/robotiq_arg2f_85_model_macro.xacro (robot description, xacro)
@@ -1,12 +1,11 @@
 <?xml version="1.0"?>
 <robot xmlns:xacro="http://ros.org/wiki/xacro">
-<!--  <xacro:include filename="$(find robotiq_2f_85_gripper_visualization)/urdf/robotiq_arg2f_transmission.xacro" />-->
   <xacro:macro name="outer_knuckle" params="prefix fingerprefix stroke">
     <link name="${prefix}${fingerprefix}_outer_knuckle">
-      <!--<inertial>
+      <inertial>
         <origin xyz="-0.000200000000003065 0.0199435877845359 0.0292245259211331" rpy="0 0 0" />
         <mass value="0.00853198276973456" />
         <inertia ixx="2.89328108496468E-06" ixy="-1.57935047237397E-19" ixz="-1.93980378593255E-19" iyy="1.86719750325683E-06" iyz="-1.21858577871576E-06" izz="1.21905238907251E-06" />
-        </inertial> -->
+        </inertial>
       <visual>
         <origin xyz="0 0 0" rpy="0 0 0" />
@@ -28,9 +27,9 @@
   <xacro:macro name="outer_finger" params="prefix fingerprefix stroke">
     <link name="${prefix}${fingerprefix}_outer_finger">
-      <!--<inertial>
+      <inertial>
         <origin xyz="0.00030115855001899 0.0373907951953854 -0.0208027427000385" rpy="0 0 0" />
         <mass value="0.022614240507152" />
         <inertia ixx="1.52518312458174E-05" ixy="9.76583423954399E-10" ixz="-5.43838577022588E-10" iyy="6.17694243867776E-06" iyz="6.78636130740228E-06" izz="1.16494917907219E-05" />
-        </inertial> -->
+        </inertial>
       <visual>
         <origin xyz="0 0 0" rpy="0 0 0" />
@@ -52,9 +51,9 @@
   <xacro:macro name="inner_knuckle" params="prefix fingerprefix stroke">
     <link name="${prefix}${fingerprefix}_inner_knuckle">
-      <!--<inertial>
+      <inertial>
         <origin xyz="0.000123011831763771 0.0507850843201817 0.00103968640075166" rpy="0 0 0" />
        <mass value="0.0271177346495152" />
         <inertia ixx="2.61910379223783E-05" ixy="-2.43616858946494E-07" ixz="-6.37789906117123E-09" iyy="2.8270243746167E-06" iyz="-5.37200748039765E-07" izz="2.83695868220296E-05" />
-        </inertial> -->
+        </inertial>
       <visual>
         <origin xyz="0 0 0" rpy="0 0 0" />
@@ -76,9 +75,9 @@
   <xacro:macro name="inner_finger" params="prefix fingerprefix stroke">
     <link name="${prefix}${fingerprefix}_inner_finger">
-      <!--<inertial>
+      <inertial>
         <origin xyz="0.000299999999999317 0.0160078233491243 -0.0136945669206257" rpy="0 0 0" />
         <mass value="0.0104003125914103" />
         <inertia ixx="2.71909453810972E-06" ixy="1.35402465472579E-21" ixz="-7.1817349065269E-22" iyy="7.69100314106116E-07" iyz="6.74715432769696E-07" izz="2.30315190420171E-06" />
-        </inertial> -->
+        </inertial>
       <visual>
         <origin xyz="0 0 0" rpy="0 0 0" />
@@ -187,5 +186,4 @@
     <xacro:finger_joint prefix="${prefix}"/>
     <xacro:right_outer_knuckle_joint prefix="${prefix}"/>
-<!--    <xacro:robotiq_arg2f_transmission prefix="${prefix}"/>-->
   </xacro:macro>
 </robot>

File: robotiq_2f_85_gripper_visualization/urdf/robotiq_gripper.urdf.xacro (robot description, xacro)
@@ -4,13 +4,26 @@
     <xacro:arg name="fake_sensor_commands" default="false" />
     <xacro:arg name="prefix" default="" />
+    <xacro:arg name="sim_ignition" default="false" />
     <!-- Import macros -->
     <xacro:include filename="$(find robotiq_2f_85_gripper_visualization)/urdf/robotiq_arg2f_85_model_macro.xacro" />
     <xacro:include filename="$(find robotiq_2f_85_gripper_visualization)/urdf/robotiq_gripper.ros2_control.xacro" />
-<!--    <link name="world" />-->
+    <link name="world" />
+    <joint name="world_to_base" type="fixed">
+        <origin rpy="0 0 0" xyz="0 0 0"/>
+        <parent link="world"/>
+        <child link="$(arg prefix)robotiq_arg2f_base_link"/>
+    </joint>
     <xacro:robotiq_arg2f_85 prefix="$(arg prefix)"/>
     <xacro:robotiq_sim_gripper_ros2_control name="RobotiqGripperSystem"
                                             prefix="$(arg prefix)"
-                                            sim_ignition="false"
+                                            sim_ignition="$(arg sim_ignition)"
                                             use_fake_hardware="$(arg use_fake_hardware)"
                                             fake_sensor_commands="$(arg fake_sensor_commands)" />
+    <xacro:if value="$(arg sim_ignition)">
+        <gazebo>
+            <plugin filename="ign_ros2_control-system" name="ign_ros2_control::IgnitionROS2ControlPlugin">
+                <parameters>$(find robotiq_bringup)/config/robotiq_2f_85_controllers.yaml</parameters>
+            </plugin>
+        </gazebo>
+    </xacro:if>
 </robot>

Commit message: Fix limits and dynamics.

File: robotiq_2f_85_gripper_visualization/urdf/robotiq_arg2f_85_model_macro.xacro (robot description, xacro)
@@ -136,4 +136,5 @@
       <axis xyz="1 0 0" />
       <limit lower="0" upper="0.8757" velocity="2.0" effort="1000" />
+      <dynamics damping="0.5" />
       <mimic joint="${prefix}finger_joint" multiplier="1" offset="0" />
     </joint>
@@ -145,5 +146,6 @@
       <child link="${prefix}${fingerprefix}_inner_finger" />
       <axis xyz="1 0 0" />
-      <limit lower="0" upper="0.8757" velocity="2.0" effort="1000" />
+      <limit lower="-0.8757" upper="0.0" velocity="2.0" effort="1000" />
+      <dynamics damping="0.5" />
       <mimic joint="${prefix}finger_joint" multiplier="-1" offset="0" />
     </joint>
@@ -165,4 +167,5 @@
       <axis xyz="1 0 0" />
       <limit lower="0" upper="0.8" velocity="2.0" effort="1000" />
+      <dynamics damping="0.5" />
     </joint>
     <xacro:finger_joints prefix="${prefix}" fingerprefix="left" reflect="1.0"/>
@@ -175,4 +178,5 @@
       <axis xyz="1 0 0" />
       <limit lower="0" upper="0.81" velocity="2.0" effort="1000" />
+      <dynamics damping="0.5" />
       <mimic joint="${prefix}finger_joint" multiplier="1" offset="0" />
     </joint>

Commit message: Adapt i term for finger joint. Remove collision for inner knuckle.

File: robotiq_2f_85_gripper_visualization/urdf/robotiq_arg2f_85_model_macro.xacro (robot description, xacro)
@@ -90,15 +90,15 @@
         </material>
       </visual>
-      <collision>
-        <origin xyz="0 0 0" rpy="0 0 0" />
-        <geometry>
-          <xacro:if value="${force_abs_paths}">
-            <mesh filename="file://$(find robotiq_2f_85_gripper_visualization)/meshes/collision/robotiq_arg2f_85_inner_knuckle.dae" scale="0.001 0.001 0.001"/>
-          </xacro:if>
-          <xacro:unless value="${force_abs_paths}">
-            <mesh filename="package://robotiq_2f_85_gripper_visualization/meshes/collision/robotiq_arg2f_85_inner_knuckle.dae" scale="0.001 0.001 0.001"/>
-          </xacro:unless>
-        </geometry>
-      </collision>
+<!--      <collision>-->
+<!--        <origin xyz="0 0 0" rpy="0 0 0" />-->
+<!--        <geometry>-->
+<!--          <xacro:if value="${force_abs_paths}">-->
+<!--            <mesh filename="file://$(find robotiq_2f_85_gripper_visualization)/meshes/collision/robotiq_arg2f_85_inner_knuckle.dae" scale="0.001 0.001 0.001"/>-->
+<!--          </xacro:if>-->
+<!--          <xacro:unless value="${force_abs_paths}">-->
+<!--            <mesh filename="package://robotiq_2f_85_gripper_visualization/meshes/collision/robotiq_arg2f_85_inner_knuckle.dae" scale="0.001 0.001 0.001"/>-->
+<!--          </xacro:unless>-->
+<!--        </geometry>-->
+<!--      </collision>-->
     </link>
   </xacro:macro>
@@ -175,5 +175,5 @@
       <child link="${prefix}${fingerprefix}_inner_knuckle" />
       <axis xyz="1 0 0" />
-      <limit lower="0" upper="0.8757" velocity="2.0" effort="1000" />
+      <limit lower="0" upper="0.8757" velocity="0.5" effort="1000" />
       <dynamics damping="3.0" />
       <mimic joint="${prefix}finger_joint" multiplier="1" offset="0" />
@@ -186,5 +186,5 @@
       <child link="${prefix}${fingerprefix}_inner_finger" />
       <axis xyz="1 0 0" />
-      <limit lower="-0.8757" upper="0.0" velocity="2.0" effort="1000" />
+      <limit lower="-0.8757" upper="0.0" velocity="0.5" effort="1000" />
       <dynamics damping="3.0" />
       <mimic joint="${prefix}finger_joint" multiplier="-1" offset="0" />
@@ -206,5 +206,5 @@
       <child link="${prefix}left_outer_knuckle" />
       <axis xyz="1 0 0" />
-      <limit lower="0" upper="0.8" velocity="2.0" effort="1000" />
+      <limit lower="0" upper="0.8" velocity="0.5" effort="1000" />
       <dynamics damping="3.0" />
     </joint>
@@ -217,5 +217,5 @@
       <child link="${prefix}right_outer_knuckle" />
       <axis xyz="1 0 0" />
-      <limit lower="0" upper="0.81" velocity="2.0" effort="1000" />
+      <limit lower="0" upper="0.81" velocity="0.5" effort="1000" />
       <dynamics damping="3.0" />
       <mimic joint="${prefix}finger_joint" multiplier="1" offset="0" />

File: robotiq_2f_85_gripper_visualization/urdf/robotiq_gripper.ros2_control.xacro (robot description, xacro)
@@ -30,9 +30,9 @@
                 <param name="cmdMin_pos">-2.0</param>
                 <param name="cmdOffset_pos">0.0</param>
-                <param name="p_vel">500.0</param>
-                <param name="i_vel">1.0</param>
+                <param name="p_vel">100.0</param>
+                <param name="i_vel">100.0</param>
                 <param name="d_vel">0.0</param>
-                <param name="iMax_vel">1.0</param>
-                <param name="iMin_vel">-1.0</param>
+                <param name="iMax_vel">100.0</param>
+                <param name="iMin_vel">-100.0</param>
                 <param name="cmdMax_vel">1000.0</param>
                 <param name="cmdMin_vel">-1000.0</param>
@@ -55,5 +55,5 @@
                 <param name="p_vel">100.0</param>
                 <param name="i_vel">1.0</param>
-                <param name="d_vel">0.0</param>
+                <param name="d_vel">0.1</param>
                 <param name="iMax_vel">50.0</param>
                 <param name="iMin_vel">-50.0</param>
